File: Leonardo_Rev3d.kicad_pcb (KiCad board)
At the start: 2 copper layers, 68.6 x 53.3 mm, 60 parts, among them IC1 NCP1117ST50T3G, IC2 LMV358IDGKR, J1 USB Micro, J2 8x1F-H8.5, J3 8x1F-H8.5, J4 6x1F-H8.5, T1 FDN340P, U1 ATMEGA32U4-XUMU, U2 ATMEGA32U4-XUAU, U3 LP2985-33DBVR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

Commit message: update version
Parts:
- added JP2: OTG, Leonardo_Rev3d:HEADER_2_2.54, F.Cu at (118.5, 86.8)
- D2: value CD1206-S01575 -> 1N4148W-TP
- J1: value USB Micro -> USBMICRO; footprint Leonardo_Rev3d:CON2_USB_MICRO_B_AT_OVAL -> Leonardo_Rev3d:10118194-0001LF
- RESET0: renamed from RESET; value TS42 -> >VALUE; footprint Leonardo_Rev3d:TS42 -> Leonardo_Rev3d:TS07
- moved GND0 1.27 mm to (120.7, 96.1)
- moved J1 0.37 mm to (116.0, 93.6)
Connections:
- net +3V3 renamed /+3V3
- net A0 renamed /A0
- net A1 renamed /A1
- net A2 renamed /A2
- net A3 renamed /A3
- net A4 renamed /A4
- net A5 renamed /A5
- net AGND renamed /AGND
- net AREF renamed /AREF
- net CMP renamed /CMP
- net D+ renamed /D+
- net D- renamed /D-
- net D0/RX renamed /D0/RX
- net D1/TX renamed /D1/TX
- net D2/SDA renamed /D2/SDA
- net D3/SCL renamed /D3/SCL
- net D4 renamed /D4
- net D5* renamed /D5*
- net D6* renamed /D6*
- net GATE_CMD renamed /GATE_CMD
- net IO10* renamed /IO10*
- net IO11* renamed /IO11*
- net IO12 renamed /IO12
- net IO13* renamed /IO13*
- net IO8 renamed /IO8
- net IO9* renamed /IO9*
- net LL renamed /LL
- net MISO renamed /MISO
- net MOSI renamed /MOSI
- net RD+ renamed /RD+
- net RD- renamed /RD-
- net RXLED renamed /RXLED
- net SCK renamed /SCK
- net TXLED renamed /TXLED
- net UCAP renamed /UCAP
- net UGND renamed GND1
- net VIN renamed /VIN
- net XTAL1 renamed /XTAL1
- net XTAL2 renamed /XTAL2
- net XUSB renamed /XUSB
- C1 pad 2: GND -> COM
- C10 pad -: GND -> COM
- C11 pad 1: GND -> COM
- C12 pad -: GND -> COM
- C13 pad 2: GND -> COM
- C14 pad 1: GND -> COM
- C2 pad 2: GND -> COM
- C22 pad 1: GND -> COM
- C3 pad 1: GND -> COM
- C4 pad 2: GND -> COM
- C5 pad 1: AVCC -> +5V
- C5 pad 2: GND -> COM
- C8 pad -: GND -> COM
- C9 pad 1: GND -> COM
- D1 pad A: GND -> COM
- D2 pad A: RESET -> /RESET
- EXTPOWER0 pad 1: GND -> COM
- EXTPOWER0 pad 3: GND -> COM
- GND0 pad X: GND -> COM
- IC1 pad 1: GND -> COM
- IC2 pad 4: GND -> COM
- ICSP0 pad 5: RESET -> /RESET
- ICSP0 pad 6: GND -> COM
- J1 pad P4: USBID -> /USBID
- J1 pad S5: GND -> (no net)
- J1 pad S6: GND -> (no net)
- J2 pad 8: D7 -> /D7
- J3 pad 1: (no net) -> unconnected-(J3-Pad1)
- J3 pad 3: RESET -> /RESET
- J3 pad 6: GND -> COM
- J3 pad 7: GND -> COM
- JP1 pad 7: GND -> COM
- L0 pad C: GND -> COM
- L1 pad 2: AVCC -> +5V
- L2 pad 2: GND -> COM
- ON0 pad C: GND -> COM
- R2 pad 2: GND -> COM
- R3 pad 1: GND -> COM
- R4 pad 1: GND -> COM
- RESET0 pad 1: RESET -> /RESET
- RESET0 pad 2: RESET -> COM
- RESET0 pad 3: GND -> /RESET
- RESET0 pad 4: GND -> COM
- RN1 pad 2: GND -> COM
- RN1 pad 3: GND -> COM
- RN1 pad 4: RESET -> /RESET
- RN1 pad 6: HWB -> /D7
- RN3 pad 2: (no net) -> unconnected-(RN3-Pad2)
- RN3 pad 3: (no net) -> unconnected-(RN3-Pad3)
- RN3 pad 6: (no net) -> unconnected-(RN3-Pad6)
- RN3 pad 7: (no net) -> unconnected-(RN3-Pad7)
- U1 pad 1: D7 -> /D7
- U1 pad 13: RESET -> /RESET
- U1 pad 15: GND -> COM
- U1 pad 23: GND -> COM
- U1 pad 24: AVCC -> +5V
- U1 pad 33: HWB -> /D7
- U1 pad 35: GND -> COM
- U1 pad 44: AVCC -> +5V
- U1 pad EXP: GND -> COM
- U2 pad 1: D7 -> /D7
- U2 pad 13: RESET -> /RESET
- U2 pad 15: GND -> COM
- U2 pad 23: GND -> COM
- U2 pad 24: AVCC -> +5V
- U2 pad 33: HWB -> /D7
- U2 pad 35: GND -> COM
- U2 pad 44: AVCC -> +5V
- U2 pad P$1: GND -> COM
- U3 pad 2: GND -> COM
- U3 pad 4: (no net) -> unconnected-(U3-Pad4)
- Y1 pad 2: GND -> COM
- Y1 pad 4: GND -> COM
- Z1 pad 2: GND -> COM
- Z2 pad 2: GND -> COM
Routing:
- net /RESET: track 0.00 -> 189.6 mm, vias 0 -> 5
- net RESET: track 185.3 -> 0.00 mm, vias 3 -> 0
- net /D7: track 0.00 -> 101.7 mm, vias 0 -> 3
- net COM: track 0.00 -> 99.9 mm, vias 0 -> 21
- net GND: track 81.7 -> 0.00 mm, vias 22 -> 0
- net +5V: track 226.5 -> 301.0 mm, vias 18 -> 23
- net AVCC: track 73.5 -> 0.00 mm, vias 5 -> 0
- net D7: track 62.0 -> 0.00 mm, vias 3 -> 0
- net HWB: track 17.8 -> 0.00 mm
- net /USBID: track 0.00 -> 13.0 mm, vias 0 -> 1
- net /D+: track 14.3 -> 12.4 mm
- net /D-: track 12.2 -> 11.5 mm
- net GND1: track 78.5 -> 77.9 mm
- added copper zone on B.Cu, net COM
- added copper zone on F.Cu, net COM
- removed copper zone on B.Cu, net GND
- removed copper zone on F.Cu, net GND
