File: Leonardo_Rev3d.kicad_pcb (KiCad board)
At the start: 2 copper layers, 68.6 x 53.3 mm, 61 parts, among them IC1 NCP1117ST50T3G, IC2 LMV358IDGKR, J1 USBMICRO, J2 8x1F-H8.5, J3 8x1F-H8.5, J4 6x1F-H8.5, T1 FDN340P, U1 ATMEGA32U4-XUMU, U2 ATMEGA32U4-XUAU, U3 LP2985-33DBVR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

Commit message: Update documentation
Parts:
- IC1: value NCP1117ST50T3G -> REG1117-5
- RESET0: value >VALUE -> TS07-667-30-BK-160-SMT-TR
