File: Leonardo_Rev3d.kicad_sch (KiCad schematic)
At the start: 55 parts, among them IC1 NCP1117ST50T3G, IC2 LMV358IDGKR, J1 USB Micro, J2 8x1F-H8.5, J3 8x1F-H8.5, J4 6x1F-H8.5, T1 FDN340P, U1 ATMEGA32U4-XUMU, U2 ATMEGA32U4-XUAU, U3 LP2985-33DBVR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

Commit message: update version
Parts:
- removed J1: USB Micro, Leonardo_Rev3d:CON2_USB_MICRO_B_AT, symbol Leonardo_Rev3d:USB-MICRO-LEGACY
- added J1: USBMICRO, Leonardo_Rev3d:10118194-0001LF, symbol Leonardo_Rev3d:USBMICRO
- added JP2: OTG, Leonardo_Rev3d:HEADER_2_2.54, symbol Leonardo_Rev3d:Jumper_2_Open
- RESET0: value TS42 -> TS07-667-30-BK-160-SMT-TR; footprint Leonardo_Rev3d:TS42 -> Leonardo_Rev3d:TS07; symbol Leonardo_Rev3d:TS42 -> Leonardo_Rev3d:TS07
Connections:
- net COM: now also RESET0.2, JP2.2 (B); no longer RESET0.3
- net D+: now also J1.P3 (D+)
- net D-: now also J1.P2 (D-)
- net GND1: now also J1.P5 (GND)
- net RESET: now also RESET0.3; no longer RESET0.2
- net USBID: now also J1.P4 (ID), JP2.1 (A)
- net XUSB: now also J1.P1 (VBUS)
Other:
- moved on the sheet: D+0

Commit message: Update documentation
Parts:
- C1, C13, C2, C22, C6, C9: Digikey_ref C0603C104J4RAC7867 -> 399-C0603C104J4RAC7867CT-ND; Manufacturer (none) -> Kemet; Manufacturer_ref (none) -> C0603C104J4RAC7867
- C10, C12, C8: Digikey_ref (none) -> 399-3708-1-ND; Manufacturer (none) -> Kemet; Manufacturer_ref (none) -> T491B106M016AT
- C11, C14, C5, C7: Digikey_ref C0603C104J4RAC7867 -> 399-C0603C105K4RAC7411CT-ND; Manufacturer (none) -> Kemet; Manufacturer_ref (none) -> C0603C105K4RAC7411
- C3, C4: Digikey_ref C0603C104J4RAC7867 -> 399-14962-1-ND; Manufacturer (none) -> Kemet; Manufacturer_ref (none) -> C0603C220K5RAC7867
- D2: Digikey_ref (none) -> 1N4148WTPMSCT-ND; Manufacturer (none) -> MCC; Manufacturer_ref (none) -> 1N4148W-TP
- F1: Digikey_ref (none) -> MF-MSMF050-2CT-ND; Manufacturer (none) -> Bourns; Manufacturer_ref (none) -> MF-MSMF050-2
- IC1: value NCP1117ST50T3G -> REG1117-5; Digikey_ref (none) -> REG1117-5-ND; Manufacturer (none) -> TI; Manufacturer_ref (none) -> REG1117-5
- IC2: Digikey_ref (none) -> LMV358IDGKR; Manufacturer (none) -> TI; Manufacturer_ref (none) -> 296-13455-1-ND
- ICSP0: Digikey_ref (none) -> A128860-ND; Manufacturer (none) -> TE; Manufacturer_ref (none) -> 5-146486-3
- J1: Digikey_ref (none) -> 609-4618-1-ND; Manufacturer (none) -> Amphenol; Manufacturer_ref (none) -> 10118194-0001LF
- J2, J3: Digikey_ref (none) -> S7041-ND; Manufacturer (none) -> Sullins; Manufacturer_ref (none) -> PPPC081LFBN-RC
- J4: Digikey_ref (none) -> S7039-ND; Manufacturer (none) -> Sullins; Manufacturer_ref (none) -> PPPC061LFBN-RC
- JP1: Digikey_ref (none) -> S7043-ND; Manufacturer (none) -> Sullins; Manufacturer_ref (none) -> PPPC101LFBN-RC
- JP2: Digikey https://www.digikey.fr/fr/products/detail/samtec-inc/DW-02-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 -> (none); Digikey_ref (none) -> SAM15134-ND; Manufacturer (none) -> Samtex; Manufacturer_ref (none) -> DW-02-07-T-S-200
- L0: Digikey_ref (none) -> 160-1428-1-ND; Manufacturer (none) -> Lite-on; Manufacturer_ref (none) -> LTST-C171KSKT
- L1, L2: Digikey_ref (none) -> MH2029-300YCT-ND; Manufacturer (none) -> Bourns; Manufacturer_ref (none) -> MH2029-300Y
- ON0: Digikey_ref (none) -> 160-1426-1-ND; Manufacturer (none) -> Lite-on; Manufacturer_ref (none) -> LTST-C171KGKT
- R1: Digikey_ref (none) -> CR0603-FX-1004ELFCT-ND; Manufacturer (none) -> Bourns; Manufacturer_ref (none) -> CR0603-FX-1004ELF
- R4: Digikey_ref (none) -> CR0603-FX-1002ELFCT-ND; Manufacturer (none) -> Bourns; Manufacturer_ref (none) -> CR0603-FX-1002ELF
- RESET0: Digikey_ref (none) -> 2223-TS07-667-30-BK-160-SMT-TRCT-ND; Manufacturer (none) -> CUI; Manufacturer_ref (none) -> TS07-667-30-BK-160-SMT-TR
- RN1: Digikey_ref (none) -> CAY16-1002F4LFCT-ND; Manufacturer (none) -> Bourns; Manufacturer_ref (none) -> CAY16-1002F4LF
- RN2: Digikey_Ref CAY16-1001F4LF -> (none); Digikey_ref (none) -> CAY16-1001F4LFCT-ND; Manufacturer (none) -> Bourns; Manufacturer_ref (none) -> CAY16-1001F4LF
- RN3: DigiKeyRef CAY16-22R0F4LF -> (none); Digikey_ref (none) -> CAY16-22R0F4LFCT-ND; Manufacturer (none) -> Bourns; Manufacturer_ref (none) -> CAY16-22R0F4LF
- RX0, TX0: Digikey_ref (none) -> 160-1426-1-ND; Manufacturer (none) -> Lite-on; Manufacturer_ref (none) -> LTST-C171KSKT
- T1: Digikey_ref (none) -> 4518-FDN340PCT-ND; Manufacturer (none) -> UMW; Manufacturer_ref (none) -> FDN340P
- U1: Digikey_ref (none) -> ATMEGA32U4-MU-ND; Manufacturer (none) -> Microchip; Manufacturer_ref (none) -> ATMEGA32U4-MU
- U2: Digikey_ref (none) -> ATMEGA32U4-AU-ND; Manufacturer (none) -> Microchip; Manufacturer_ref (none) -> ATMEGA32U4-AU
- U3: Digikey_ref (none) -> LP2985IM5-3.3CT-ND; Manufacturer (none) -> TI; Manufacturer_ref (none) -> LP2985IM5-3.3
- Z1, Z2: Digikey_ref (none) -> CG0603MLC-05ECT-ND; Manufacturer (none) -> Bourns; Manufacturer_ref (none) -> CG0603MLC-05E
