File: Leonardo_Rev3e.kicad_pcb (KiCad board)
At the start: 2 copper layers, 68.6 x 53.3 mm, 61 parts, among them IC1 REG1117-5, IC2 LMV358IDGKR, J1 USBMICRO, J2 8x1F-H8.5, J3 8x1F-H8.5, J4 6x1F-H8.5, T1 FDN340P, U1 ATMEGA32U4-XUMU, U2 ATMEGA32U4-XUAU, U3 LP2985-33DBVR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

Commit message: feat: add labels to match original design
Other:
- board text added: "ICSP"
- board text added: "L"
- board text added: "ON"
- board text added: "RESET"
- board text added: "RX"
- board text added: "TX"
